Commit message: Correct lidar frame

File: config/urdf/RSBPearl_raysim.urdf.xacro (robot description, xacro)
@@ -6,7 +6,7 @@
       <xacro:insert_block name="origin" />
       <parent link="${parent}"/>
-      <child link="${name}_base_link"/>
+      <child link="${name}"/>
     </joint>
-    <link name="${name}_base_link">
+    <link name="${name}">
       <inertial>
         <mass value="0.83"/>
@@ -21,16 +21,4 @@
         </geometry>
       </visual>
-    </link>
-    <joint name="${name}_base_scan_joint" type="fixed" >
-      <origin xyz="0 0 0.0377" rpy="0 0 0" />
-      <parent link="${name}_base_link" />
-      <child link="${name}"/>
-    </joint>
-    <link name="${name}">
-      <inertial>
-        <mass value="0.01"/>
-        <origin xyz="0 0 0"/>
-        <inertia ixx="1e-7" ixy="0" ixz="0" iyy="1e-7" iyz="0" izz="1e-7"/>
-      </inertial>
     </link>
     <!-- Gazebo requires the velodyne_gazebo_plugins package -->

File: config/urdf/example.urdf.xacro (robot description, xacro)
@@ -39,5 +39,5 @@
     </link>
     <xacro:include filename="$(find rslidar_sdk)/config/urdf/RSBPearl_raysim.urdf.xacro"/>
-    <xacro:RSBPearl_raysim parent="base_rslidar" name="rslidar" topic="/rslidar_points" hz="10" samples="1800" gpu="${gpu}">
+    <xacro:RSBPearl_raysim parent="base_rslidar" name="rslidar_optical_center" topic="/rslidar_points" hz="10" samples="1800" gpu="${gpu}">
       <origin xyz="0 0 0" rpy="0 0 0" />
     </xacro:RSBPearl_raysim>
